File: Reprap LCD Click/RLC.sch (EAGLE design)
At the start: 10 parts, among them IC1 PCF8574T, Q1 BC548B, SW1 EC12E_SW, X1 HD44780LCD-1602

Commit message: r1v3, reprap LCD clicker, alvin board
Parts:
- removed QUAD: (no value), con-lstb:MA03-1
- removed R1: (no value), rcl:POTENTIOMETER_PT-10
- removed SW1: EC12E_SW, switch-alps:EC12E_SW
- added R2: (no value), pot:TRIM_EU-CA6V
Connections:
- removed net N$15: QUAD.3, SW1G$2.2
- removed net N$16: QUAD.2, SW1G$1.B
- removed net N$17: QUAD.1, SW1G$1.A
- net +5V: now also R2.E; no longer R1.2
- net GND: now also R2.A; no longer R1.1, SW1G$1.C, SW1G$2.1
- net N$13: now also R2.S; no longer R1.3
